File: kicad/temp-measurements/temp-measurements.kicad_sch (KiCad schematic)
At the start: 31 parts, among them U1 LM324, U2 Arduino_pro_mini, U3 LM431

Commit message: commiting all uncommited, clean up
Parts:
- removed R12: 2.74k, Resistor_SMD:R_1206_3216Metric_Pad1.30x1.75mm_HandSolder, symbol Device:R_US
- removed R13: 3.32k, Resistor_SMD:R_1206_3216Metric_Pad1.30x1.75mm_HandSolder, symbol Device:R_US
- removed RV1, RV2: 10k, symbol Device:R_Potentiometer_US
- removed U2: Arduino_pro_mini, !my-kicad-library:ARDUINO_PRO_MINI_NO_A5, symbol !my-kicad-library:Arduino_pro_mini
- added C7: 10u+, symbol Device:C_Polarized_US
- added D1, D2: BAT54S, Package_TO_SOT_SMD:SOT-23, symbol Diode:BAT54S
- added J1: FAN, symbol Connector:Conn_01x02_Male
- added Q1: 2N7000, Package_TO_SOT_THT:TO-92_Inline, symbol Transistor_FET:2N7000
- added R14, R15, R16, R17, R18: 10k, Resistor_SMD:R_1206_3216Metric_Pad1.30x1.75mm_HandSolder, symbol Device:R_US
- added U4: Arduino_nano_narrow, !my-kicad-library:ARDUINO_NANO_NARROW, symbol !my-kicad-library:Arduino_nano_narrow
- added U?: LM431, Package_TO_SOT_THT:TO-92L_HandSolder, symbol !my-kicad-library:LM431
- gave numbers to parts that had none: 7
Connections:
- net temp1 is gone; now on net TEMP1: R9.2, U1.7
- net temp2 is gone; now on net TEMP2: R10.2, U1.14
- net 5V: now also C7.1, D1.2, D2.2, U4.5V
- net GND: now also C7.2, D1.1, D2.1, Q1.1 (S), R15.2, R17.2, R18.2, U4.GND, U?.2 (A); no longer U3.2 (A)
- net TEMP1: now also D1.3, U4.A0
- net TEMP2: now also D2.3, U4.A1
- net V_IN: now also J1.1 (Pin_1)
- net V_REF: now also U3.1 (REF), R14.1, R16.1, U4.VREF
- net at R5.1: now also R14.2, R15.1
- net at R6.1: now also R16.2, R17.1
- new net: J1.2 (Pin_2), Q1.3 (D)
- new net: U3.2 (A), U?.1 (REF), U?.3 (K)
- new net FAN_PWM: Q1.2 (G), R18.1, U4.5
- new net SDA: U4.A4
- new net SLC: U4.A5
- no-connect marks 13 -> 21
Other:
- note added: "5V (measure actual voltage and set in firmware) 10mA available"
- note added: "Voltage reference"
- note added: "opamp offsets and x10 voltage"
- note added: "remote wire sensor"
- note added: "second heatsink/IC"
- note added: "temperature measurement"
- note removed: "adjust to shift voltage down ~2.275V"
- note removed: "figure out aref pin"
- note removed: "~4.55V 10mA available"
- moved on the sheet: C6, R1, R10, R11, R2, R3, R4, R5, R6, R7, R8, R9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
